File: Hardware/Electronics/ePaperShoe/ScreenCircuitV0.2.brd (EAGLE design)
At the start: 22.8 x 36.5 mm, 15 parts, among them Q1 IRF7509, U1 XF2J-2624-11A, X1 FH12-26S-0.5SH

Commit message: Made screen circuit version 0.2
Parts:
- removed D1, D2: 120mA/40V/370mV, SparkFun-DiscreteSemi:SOD-523
- added D3, D4: 0.5A/40V/420mV, SparkFun-DiscreteSemi:SOD-323
- moved C3 1.08 mm to (19.8, 21.1)
- moved C6 0.92 mm to (11.9, 21.1)
- moved C4 0.92 mm to (15.7, 21.1)
- moved C2 0.76 mm to (19.8, 27.9)
- moved Q1 0.76 mm to (3.05, 20.3)
- moved C5 0.57 mm to (2.29, 8.89)
- moved C7 0.51 mm to (11.9, 27.9)
- moved U1 0.51 mm to (5.08, 9.65)
- moved C1 0.51 mm to (15.7, 27.9)
Connections:
- net N$3: now also D3.C; no longer D1.C
- net N$5: now also D4.A; no longer D2.A
- net VGH: now also D4.C; no longer D2.C
- net VGL: now also D3.A; no longer D1.A
Routing:
- net SPI_MISO: track 63.2 -> 39.0 mm, vias 1 -> 2
- net SPI_CS: track 51.0 -> 28.2 mm
- net SPI_MOSI: track 46.2 -> 30.2 mm, vias 0 -> 1
- net VGH: track 35.8 -> 48.1 mm, vias 2 -> 3
- net 3.3V: track 73.1 -> 84.5 mm, vias 4 -> 2
- net SPI_CLK: track 32.1 -> 43.3 mm, vias 1 -> 2
- net GDR_N: track 33.4 -> 24.7 mm, vias 3 -> 0
- net GND: track 110.7 -> 118.9 mm, vias 5 -> 0
- net RST_N: track 35.5 -> 32.2 mm, vias 0 -> 2
- net VSL: track 21.2 -> 24.1 mm
- net VDD: track 30.1 -> 32.9 mm, vias 3 -> 4
- net GDR_P: track 20.1 -> 22.6 mm
- net N$3: track 15.6 -> 16.9 mm
- net VSH: track 12.8 -> 13.8 mm
- net VGL: track 30.9 -> 30.3 mm
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- added copper zone on layer 16, net GND
- added copper zone on layer 1, net N$1
Other:
- board text added: "Bioworld ePaper shoe screen driver board V1.1"
- board text added: "V1.1"
- board text removed: "Bioworld ePaper shoe screen driver board V1.0"
- board text removed: "V1.0"
